File: ECE477.kicad_pcb (KiCad board)
At the start: 2 copper layers, 53 parts, among them IC1 LP3852EMP-3.3_NOPB, IC2 BQ29330DBT, J1 P7805-2000-S, J2 Conn_01x05_Male, J3 Conn_01x05_Male, J4 Conn_01x05_Male, J5 Conn_01x05_Male, J6 Conn_01x05_Male, SW1 SW_Push_Dual, U1 STM32H7_LQFP144_T2

Commit message: Working with Routing
Parts:
- added J7: Conn_01x05_Male, Connector_PinHeader_1.00mm:PinHeader_1x05_P1.00mm_Vertical, F.Cu at (133.3, 3.57)
- added R10: 0R, Resistor_SMD:R_0805_2012Metric_Pad1.15x1.40mm_HandSolder, F.Cu at (142.1, 6.47)
- added R6: 0R, Resistor_SMD:R_0805_2012Metric_Pad1.15x1.40mm_HandSolder, F.Cu at (137.3, 3.52)
- added R7: 0R, Resistor_SMD:R_0805_2012Metric_Pad1.15x1.40mm_HandSolder, F.Cu at (137.3, 6.47)
- added R8: 0R, Resistor_SMD:R_0805_2012Metric_Pad1.15x1.40mm_HandSolder, F.Cu at (142.1, 3.52)
- added R9: 0R, Resistor_SMD:R_0805_2012Metric_Pad1.15x1.40mm_HandSolder, F.Cu at (137.3, 9.42)
- moved J6 73.3 mm to (224.8, 44.5)
- moved IC2 62.3 mm to (234.9, 45.7)
Connections:
- net 3.3V renamed 3.3_VDD
- net 3V3_PER renamed 3V3_VDD
- C1 pad 1: VDDSMPS_IN -> VBAT
- C10 pad 1: VDDSMPS_IN -> VBAT
- C11 pad 1: VDDSMPS_IN -> VBAT
- C12 pad 1: VDDSMPS_IN -> VBAT
- C13 pad 1: VDDSMPS_IN -> VBAT
- C14 pad 1: VDDSMPS_IN -> VBAT
- C16 pad 2: GND -> GNDA
- C17 pad 2: GND -> GNDA
- C18 pad 2: GND -> GNDA
- C19 pad 2: GND -> GNDA
- C2 pad 1: VDDSMPS_IN -> VBAT
- C20 pad 1: VDDSMPS_IN -> VBAT
- C21 pad 1: VDDSMPS_IN -> VBAT
- C23 pad 1: 1V2_MCU -> VDD_SMPS_IND_OUT
- C24 pad 1: 1V2_MCU -> VDD_LDO
- C25 pad 1: 1V2_MCU -> VDD_LDO
- C26 pad 1: 1V2_MCU -> VCAP
- C27 pad 1: 1V2_MCU -> VCAP
- C3 pad 1: VDDSMPS_IN -> VBAT
- C4 pad 1: VDDSMPS_IN -> VBAT
- C5 pad 1: VDDSMPS_IN -> VBAT
- C6 pad 1: VDDSMPS_IN -> VBAT
- C7 pad 1: VDDSMPS_IN -> VBAT
- C8 pad 1: VDDSMPS_IN -> VBAT
- C9 pad 1: VDDSMPS_IN -> VBAT
- IC2 pad 1: GND -> CELL-
- IC2 pad 13: Net-(IC2-Pad13) -> PWR_IN
- IC2 pad 14: Net-(IC2-Pad14) -> NC
- IC2 pad 15: Net-(IC2-Pad15) -> NC
- IC2 pad 16: Net-(IC2-Pad16) -> NC
- IC2 pad 17: Net-(IC2-Pad17) -> PWR_IN
- IC2 pad 18: Net-(IC2-Pad18) -> NC
- IC2 pad 19: Net-(IC2-Pad19) -> PWR_IN
- IC2 pad 2: PWR_IN -> CELL+
- IC2 pad 20: Net-(IC2-Pad20) -> NC
- IC2 pad 21: Net-(IC2-Pad21) -> NC
- IC2 pad 22: Net-(IC2-Pad22) -> NC
- IC2 pad 23: Net-(IC2-Pad23) -> GND
- IC2 pad 24: Net-(IC2-Pad24) -> NC
- IC2 pad 25: Net-(IC2-Pad25) -> NC
- IC2 pad 26: Net-(IC2-Pad26) -> NC
- IC2 pad 27: Net-(IC2-Pad27) -> NC
- IC2 pad 3: Net-(IC2-Pad3) -> NC
- IC2 pad 4: Net-(IC2-Pad4) -> GND
- IC2 pad 5: Net-(IC2-Pad5) -> NC
- IC2 pad 6: Net-(IC2-Pad6) -> NC
- IC2 pad 7: Net-(IC2-Pad7) -> NC
- JP1 pad 1: OFF -> GND
- JP1 pad 2: VDDSMPS_IN -> VBAT
- L1 pad 2: 1V2_MCU -> VDD_SMPS_IND_OUT
- R1 pad 1: VDDSMPS_IN -> VBAT
- R11 pad 1: 1V2_MCU -> VCAP
- R3 pad 2: VDDSMPS_IN -> VBAT
- U1 pad 1: Net-(U1-Pad1) -> NC
- U1 pad 10: Net-(U1-Pad10) -> NC
- U1 pad 100: Net-(U1-Pad100) -> NC
- U1 pad 101: Net-(U1-Pad101) -> NC
- U1 pad 103: 1V2_MCU -> VCAP
- U1 pad 105: 1V2_MCU -> VDD_LDO
- U1 pad 106: VDDSMPS_IN -> VBAT
- U1 pad 11: Net-(U1-Pad11) -> NC
- U1 pad 111: Net-(U1-Pad111) -> NC
- U1 pad 117: Net-(U1-Pad117) -> NC
- U1 pad 119: VDDSMPS_IN -> VBAT
- U1 pad 120: Net-(U1-Pad120) -> NC
- U1 pad 121: Net-(U1-Pad121) -> NC
- U1 pad 122: Net-(U1-Pad122) -> NC
- U1 pad 123: Net-(U1-Pad123) -> NC
- U1 pad 124: Net-(U1-Pad124) -> NC
- U1 pad 125: Net-(U1-Pad125) -> NC
- U1 pad 126: Net-(U1-Pad126) -> NC
- U1 pad 127: Net-(U1-Pad127) -> NC
- U1 pad 129: VDDSMPS_IN -> VBAT
- U1 pad 13: VDDSMPS_IN -> VBAT
- U1 pad 132: Net-(U1-Pad132) -> NC
- U1 pad 133: Net-(U1-Pad133) -> NC
- U1 pad 134: Net-(U1-Pad134) -> NC
- U1 pad 137: Net-(U1-Pad137) -> NC
- U1 pad 138: Net-(U1-Pad138) -> NC
- U1 pad 139: Net-(U1-Pad139) -> NC
- U1 pad 140: 1V2_MCU -> VCAP
- U1 pad 142: Net-(U1-Pad142) -> NC
- U1 pad 143: 1V2_MCU -> VDD_LDO
- U1 pad 144: VDDSMPS_IN -> VBAT
- U1 pad 16: VDDSMPS_IN -> VBAT
- U1 pad 19: VDDSMPS_IN -> VBAT
- U1 pad 2: Net-(U1-Pad2) -> NC
- U1 pad 20: Net-(U1-Pad20) -> NC
- U1 pad 21: Net-(U1-Pad21) -> NC
- U1 pad 22: Net-(U1-Pad22) -> NC
- U1 pad 23: Net-(U1-Pad23) -> NC
- U1 pad 24: Net-(U1-Pad24) -> NC
- U1 pad 25: Net-(U1-Pad25) -> NC
- U1 pad 26: Net-(U1-Pad26) -> NC
- U1 pad 28: Net-(U1-Pad28) -> NC
- U1 pad 29: Net-(U1-Pad29) -> NC
- U1 pad 3: Net-(U1-Pad3) -> NC
- U1 pad 30: Net-(U1-Pad30) -> NC
- U1 pad 31: Net-(U1-Pad31) -> NC
- U1 pad 32: VDDSMPS_IN -> VBAT
- U1 pad 34: GND -> GNDA
- U1 pad 37: Net-(U1-Pad37) -> NC
- U1 pad 38: Net-(U1-Pad38) -> NC
- U1 pad 39: Net-(U1-Pad39) -> NC
- U1 pad 4: Net-(U1-Pad4) -> NC
- U1 pad 40: Net-(U1-Pad40) -> NC
- U1 pad 42: VDDSMPS_IN -> VBAT
- U1 pad 43: Net-(U1-Pad43) -> NC
- U1 pad 44: Net-(U1-Pad44) -> NC
- U1 pad 45: Net-(U1-Pad45) -> NC
- U1 pad 46: Net-(U1-Pad46) -> NC
- U1 pad 47: Net-(U1-Pad47) -> NC
- U1 pad 48: Net-(U1-Pad48) -> NC
- U1 pad 49: Net-(U1-Pad49) -> NC
- U1 pad 5: Net-(U1-Pad5) -> NC
- U1 pad 50: Net-(U1-Pad50) -> NC
- U1 pad 51: Net-(U1-Pad51) -> NC
- U1 pad 52: Net-(U1-Pad52) -> NC
- U1 pad 53: Net-(U1-Pad53) -> NC
- U1 pad 54: Net-(U1-Pad54) -> NC
- U1 pad 56: VDDSMPS_IN -> VBAT
- U1 pad 57: Net-(U1-Pad57) -> NC
- U1 pad 58: Net-(U1-Pad58) -> NC
- U1 pad 59: Net-(U1-Pad59) -> NC
- U1 pad 60: Net-(U1-Pad60) -> NC
- U1 pad 61: Net-(U1-Pad61) -> NC
- U1 pad 62: Net-(U1-Pad62) -> NC
- U1 pad 63: Net-(U1-Pad63) -> NC
- U1 pad 64: Net-(U1-Pad64) -> NC
- U1 pad 65: Net-(U1-Pad65) -> NC
- U1 pad 68: 1V2_MCU -> VCAP
- U1 pad 7: VDDSMPS_IN -> VBAT
- U1 pad 70: 1V2_MCU -> VDD_LDO
- U1 pad 71: VDDSMPS_IN -> VBAT
- U1 pad 73: Net-(U1-Pad73) -> NC
- U1 pad 74: Net-(U1-Pad74) -> NC
- U1 pad 75: Net-(U1-Pad75) -> NC
- U1 pad 76: Net-(U1-Pad76) -> NC
- U1 pad 77: Net-(U1-Pad77) -> NC
- U1 pad 78: Net-(U1-Pad78) -> NC
- U1 pad 79: VDDSMPS_IN -> VBAT
- U1 pad 8: VDDSMPS_IN -> VBAT
- U1 pad 81: Net-(U1-Pad81) -> NC
- U1 pad 82: Net-(U1-Pad82) -> NC
- U1 pad 83: Net-(U1-Pad83) -> NC
- U1 pad 84: Net-(U1-Pad84) -> NC
- U1 pad 85: Net-(U1-Pad85) -> NC
- U1 pad 86: Net-(U1-Pad86) -> NC
- U1 pad 87: Net-(U1-Pad87) -> NC
- U1 pad 88: Net-(U1-Pad88) -> NC
- U1 pad 9: Net-(U1-Pad9) -> NC
- U1 pad 92: VDDSMPS_IN -> VBAT
- U1 pad 95: Net-(U1-Pad95) -> NC
- U1 pad 96: Net-(U1-Pad96) -> NC
- U1 pad 97: Net-(U1-Pad97) -> NC
Routing:
- net GND: track 0.00 -> 137.0 mm, vias 0 -> 2
- net 5V: track 0.00 -> 74.9 mm
- net PWR_IN: track 0.00 -> 53.5 mm, vias 0 -> 2
- net 3V3_VDD: track 0.00 -> 17.2 mm
- net Net-(C35-Pad1): track 0.00 -> 13.5 mm
- net V4: track 19.0 -> 7.54 mm
- net V5: track 19.2 -> 7.75 mm
- net V2: track 18.7 -> 7.32 mm
- net V1: track 19.0 -> 7.52 mm
- net V3: track 18.8 -> 7.72 mm
- net Net-(IC1-Pad4): track 0.00 -> 4.20 mm
- net Net-(IC1-Pad1): track 0.00 -> 3.36 mm

Commit message: Finshed Routing One
Parts:
- removed C24, C25: 100nF, Capacitor_SMD:C_0805_2012Metric_Pad1.15x1.40mm_HandSolder
- removed R9: 0R, Resistor_SMD:R_0805_2012Metric_Pad1.15x1.40mm_HandSolder
- added R14: 0R, Resistor_SMD:R_0805_2012Metric_Pad1.15x1.40mm_HandSolder, B.Cu at (192.8, 130.8)
- added R5: 0R, Resistor_SMD:R_0805_2012Metric_Pad1.15x1.40mm_HandSolder, F.Cu at (189.2, 128.3)
- C22, C23, C26, C27, L1, R10, R11, R6, R7: moved to B.Cu
- moved R3 138.0 mm to (223.5, 115.3)
- moved C30 136.0 mm to (236.2, 123.2)
- moved SW1 136.0 mm to (223.5, 120.7)
- moved R7 126.0 mm to (204.5, 113.0)
- moved J7 116.5 mm to (222.2, 78.7)
- moved R6 116.5 mm to (198.1, 102.9)
- moved R10 114.8 mm to (198.1, 106.7)
- moved R8 112.4 mm to (172.5, 111.8)
- moved C14 97.5 mm to (152.2, 29.2)
- moved C13 85.1 mm to (152.2, 34.3)
- moved C9 82.0 mm to (152.2, 53.3)
- moved C12 75.3 mm to (152.2, 39.4)
- moved U1 74.5 mm to (198.1, 106.7), turned to 90 degrees
- moved C11 69.4 mm to (152.2, 44.5)
- moved J4 65.6 mm to (176.5, 77.5), turned to 270 degrees
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Connections:
- C1 pad 1: VBAT -> VDD_MCU
- C10 pad 1: VBAT -> VDD_MCU
- C11 pad 1: VBAT -> VDD_MCU
- C12 pad 1: VBAT -> VDD_MCU
- C13 pad 1: VBAT -> VDD_MCU
- C14 pad 1: VBAT -> VDD_MCU
- C2 pad 1: VBAT -> VDD_MCU
- C20 pad 1: VBAT -> VDDSMPS_IN
- C21 pad 1: VBAT -> VDDSMPS_IN
- C3 pad 1: VBAT -> VDD_MCU
- C4 pad 1: VBAT -> VDD_MCU
- C5 pad 1: VBAT -> VDD_MCU
- C6 pad 1: VBAT -> VDD_MCU
- C7 pad 1: VBAT -> VDD_MCU
- C8 pad 1: VBAT -> VDD_MCU
- C9 pad 1: VBAT -> VDD_MCU
- IC2 pad 14: NC -> Net-(IC2-Pad14)
- IC2 pad 15: NC -> Net-(IC2-Pad15)
- IC2 pad 16: NC -> Net-(IC2-Pad16)
- IC2 pad 18: NC -> Net-(IC2-Pad18)
- IC2 pad 20: NC -> Net-(IC2-Pad20)
- IC2 pad 21: NC -> Net-(IC2-Pad21)
- IC2 pad 22: NC -> Net-(IC2-Pad22)
- IC2 pad 24: NC -> Net-(IC2-Pad24)
- IC2 pad 25: NC -> Net-(IC2-Pad25)
- IC2 pad 26: NC -> Net-(IC2-Pad26)
- IC2 pad 27: NC -> Net-(IC2-Pad27)
- IC2 pad 3: NC -> Net-(IC2-Pad3)
- IC2 pad 5: NC -> Net-(IC2-Pad5)
- IC2 pad 6: NC -> Net-(IC2-Pad6)
- IC2 pad 7: NC -> Net-(IC2-Pad7)
- J5 pad 2: 3.3_VDD -> 3V3_VDD
- J7 pad 3: NC -> Net-(J7-Pad3)
- J7 pad 4: NC -> Net-(J7-Pad4)
- J7 pad 5: NC -> Net-(J7-Pad5)
- JP1 pad 2: VBAT -> VDD_MCU
- R1 pad 1: VBAT -> VDD_MCU
- R10 pad 1: 1V2_MCU -> VDD_LDO
- R3 pad 2: VBAT -> VDD_MCU
- R6 pad 1: 1V2_MCU -> VDD_SMPS_IND_OUT
- U1 pad 1: NC -> Net-(U1-Pad1)
- U1 pad 10: NC -> Net-(U1-Pad10)
- U1 pad 100: NC -> Net-(U1-Pad100)
- U1 pad 101: NC -> Net-(U1-Pad101)
- U1 pad 106: VBAT -> VDD_MCU
- U1 pad 11: NC -> Net-(U1-Pad11)
- U1 pad 111: NC -> Net-(U1-Pad111)
- U1 pad 117: NC -> Net-(U1-Pad117)
- U1 pad 119: VBAT -> VDD_MCU
- U1 pad 120: NC -> Net-(U1-Pad120)
- U1 pad 121: NC -> Net-(U1-Pad121)
- U1 pad 122: NC -> Net-(U1-Pad122)
- U1 pad 123: NC -> Net-(U1-Pad123)
- U1 pad 124: NC -> Net-(U1-Pad124)
- U1 pad 125: NC -> Net-(U1-Pad125)
- U1 pad 126: NC -> Net-(U1-Pad126)
- U1 pad 127: NC -> Net-(U1-Pad127)
- U1 pad 129: VBAT -> VDD_MCU
- U1 pad 13: VBAT -> VDD_MCU
- U1 pad 132: NC -> Net-(U1-Pad132)
- U1 pad 133: NC -> Net-(U1-Pad133)
- U1 pad 134: NC -> Net-(U1-Pad134)
- U1 pad 137: NC -> Net-(U1-Pad137)
- U1 pad 138: NC -> Net-(U1-Pad138)
- U1 pad 139: NC -> Net-(U1-Pad139)
- U1 pad 142: NC -> Net-(U1-Pad142)
- U1 pad 144: VBAT -> VDD_MCU
- U1 pad 16: VBAT -> VDDSMPS_IN
- U1 pad 19: VBAT -> VDD_MCU
- U1 pad 2: NC -> Net-(U1-Pad2)
- U1 pad 20: NC -> Net-(U1-Pad20)
- U1 pad 21: NC -> Net-(U1-Pad21)
- U1 pad 22: NC -> Net-(U1-Pad22)
- U1 pad 23: NC -> Net-(U1-Pad23)
- U1 pad 24: NC -> Net-(U1-Pad24)
- U1 pad 25: NC -> Net-(U1-Pad25)
- U1 pad 26: NC -> Net-(U1-Pad26)
- U1 pad 28: NC -> Net-(U1-Pad28)
- U1 pad 29: NC -> Net-(U1-Pad29)
- U1 pad 3: NC -> Net-(U1-Pad3)
- U1 pad 30: NC -> Net-(U1-Pad30)
- U1 pad 31: NC -> Net-(U1-Pad31)
- U1 pad 32: VBAT -> VDD_MCU
- U1 pad 37: NC -> Net-(U1-Pad37)
- U1 pad 38: NC -> Net-(U1-Pad38)
- U1 pad 39: NC -> Net-(U1-Pad39)
- U1 pad 4: NC -> Net-(U1-Pad4)
- U1 pad 40: NC -> Net-(U1-Pad40)
- U1 pad 42: VBAT -> VDD_MCU
- U1 pad 43: NC -> Net-(U1-Pad43)
- U1 pad 44: NC -> Net-(U1-Pad44)
- U1 pad 45: NC -> Net-(U1-Pad45)
- U1 pad 46: NC -> Net-(U1-Pad46)
- U1 pad 47: NC -> Net-(U1-Pad47)
- U1 pad 48: NC -> Net-(U1-Pad48)
- U1 pad 49: NC -> Net-(U1-Pad49)
- U1 pad 5: NC -> Net-(U1-Pad5)
- U1 pad 50: NC -> Net-(U1-Pad50)
- U1 pad 51: NC -> Net-(U1-Pad51)
- U1 pad 52: NC -> Net-(U1-Pad52)
- U1 pad 53: NC -> Net-(U1-Pad53)
- U1 pad 54: NC -> Net-(U1-Pad54)
- U1 pad 56: VBAT -> VDD_MCU
- U1 pad 57: NC -> Net-(U1-Pad57)
- U1 pad 58: NC -> Net-(U1-Pad58)
- U1 pad 59: NC -> Net-(U1-Pad59)
- U1 pad 60: NC -> Net-(U1-Pad60)
- U1 pad 61: NC -> Net-(U1-Pad61)
- U1 pad 62: NC -> Net-(U1-Pad62)
- U1 pad 63: NC -> Net-(U1-Pad63)
- U1 pad 64: NC -> Net-(U1-Pad64)
- U1 pad 65: NC -> Net-(U1-Pad65)
- U1 pad 7: VBAT -> VDD_MCU
- U1 pad 71: VBAT -> VDD_MCU
- U1 pad 73: NC -> Net-(U1-Pad73)
- U1 pad 74: NC -> Net-(U1-Pad74)
- U1 pad 75: NC -> Net-(U1-Pad75)
- U1 pad 76: NC -> Net-(U1-Pad76)
- U1 pad 77: NC -> Net-(U1-Pad77)
- U1 pad 78: NC -> Net-(U1-Pad78)
- U1 pad 79: VBAT -> VDD_MCU
- U1 pad 81: NC -> Net-(U1-Pad81)
- U1 pad 82: NC -> Net-(U1-Pad82)
- U1 pad 83: NC -> Net-(U1-Pad83)
- U1 pad 84: NC -> Net-(U1-Pad84)
- U1 pad 85: NC -> Net-(U1-Pad85)
- U1 pad 86: NC -> Net-(U1-Pad86)
- U1 pad 87: NC -> Net-(U1-Pad87)
- U1 pad 88: NC -> Net-(U1-Pad88)
- U1 pad 9: NC -> Net-(U1-Pad9)
- U1 pad 92: VBAT -> VDD_MCU
- U1 pad 95: NC -> Net-(U1-Pad95)
- U1 pad 96: NC -> Net-(U1-Pad96)
- U1 pad 97: NC -> Net-(U1-Pad97)
Routing:
- net GND: track 137.0 -> 914.0 mm, vias 2 -> 21
- net VDD_MCU: track 0.00 -> 742.2 mm, vias 0 -> 4
- net Touch_Input: track 0.00 -> 167.1 mm, vias 0 -> 1
- net 3V3_VDD: track 17.2 -> 150.0 mm, vias 0 -> 7
- net VCAP: track 0.00 -> 77.8 mm, vias 0 -> 5
- net nJTRST: track 0.00 -> 65.2 mm, vias 0 -> 2
- net NRST: track 0.00 -> 62.9 mm, vias 0 -> 2
- net I2C2_SMBA: track 0.00 -> 57.0 mm, vias 0 -> 4
- net VDD_LDO: track 0.00 -> 56.6 mm, vias 0 -> 3
- net JTDO: track 0.00 -> 55.7 mm, vias 0 -> 4
- net I2C2_SCL: track 0.00 -> 52.0 mm, vias 0 -> 2
- net I2C2_SDA: track 0.00 -> 50.2 mm, vias 0 -> 2
- net JTMS_SWDIO: track 0.00 -> 33.5 mm, vias 0 -> 2
- net GNDA: track 0.00 -> 31.0 mm, vias 0 -> 2
- net JTDI: track 0.00 -> 29.5 mm, vias 0 -> 2
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
Commit message: updated NRST capacitor location closer to MCU
Parts:
- C30: moved to B.Cu
- moved C30 31.7 mm to (205.7, 114.3), turned to 90 degrees
- moved R7 2.54 mm to (204.5, 110.5)
Routing:
- net NRST: track 62.9 -> 53.5 mm
- net Touch_Input: track 167.1 -> 160.7 mm
- net GND: track 914.0 -> 910.1 mm
- net GNDA: track 31.0 -> 33.5 mm

Commit message: review with team
Routing:
- net NRST: track 53.5 -> 41.1 mm, vias 2 -> 1
- net PWR_IN: track 51.7 -> 55.2 mm
Changed lines of the file:
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@@
     (thickness 1.6)
     (drawings 0)
-    (tracks 803)
+    (tracks 801)
     (zones 0)
     (modules 58)
@@
   )
   (setup
-    (last_trace_width 0.25)
+    (last_trace_width 0.6096)
     (user_trace_width 0.6096)
     (trace_clearance 0.2)
@@
   (segment (start 196.85 120.65) (end 196.85 116.84) (width 0.25) (layer B.Cu) (net 5))
   (segment (start 196.85 116.84) (end 193.04 113.03) (width 0.25) (layer B.Cu) (net 5))
-  (segment (start 194.555 64.77) (end 203.445 55.88) (width 0.25) (layer F.Cu) (net 6))
-  (segment (start 203.445 55.88) (end 210.82 55.88) (width 0.25) (layer F.Cu) (net 6))
-  (segment (start 210.82 55.88) (end 213.36 53.34) (width 0.25) (layer F.Cu) (net 6))
   (segment (start 219.71 56.475) (end 219.71 57.15) (width 0.25) (layer F.Cu) (net 6))
-  (segment (start 216.575 53.34) (end 219.71 56.475) (width 0.25) (layer F.Cu) (net 6))
-  (segment (start 213.36 53.34) (end 216.575 53.34) (width 0.25) (layer F.Cu) (net 6))
-  (segment (start 194.555 66.82) (end 192.795 68.58) (width 0.25) (layer F.Cu) (net 6))
-  (segment (start 194.555 64.77) (end 194.555 66.82) (width 0.25) (layer F.Cu) (net 6))
-  (segment (start 193.22 72.91) (end 192.02 72.91) (width 0.25) (layer F.Cu) (net 6))
-  (segment (start 194.555 71.575) (end 193.22 72.91) (width 0.25) (layer F.Cu) (net 6))
-  (segment (start 194.555 64.77) (end 194.555 71.575) (width 0.25) (layer F.Cu) (net 6))
   (segment (start 243.84 63.5) (end 236.22 63.5) (width 0.6096) (layer F.Cu) (net 6))
   (segment (start 245.11 64.77) (end 243.84 63.5) (width 0.6096) (layer F.Cu) (net 6))
   (segment (start 229.87 57.15) (end 236.22 63.5) (width 0.6096) (layer F.Cu) (net 6))
   (segment (start 219.71 57.15) (end 229.87 57.15) (width 0.6096) (layer F.Cu) (net 6))
+  (segment (start 194.555 64.77) (end 194.555 63.255) (width 0.6096) (layer F.Cu) (net 6))
+  (segment (start 194.555 63.255) (end 204.47 53.34) (width 0.6096) (layer F.Cu) (net 6))
+  (segment (start 219.71 56.1154) (end 219.71 57.15) (width 0.6096) (layer F.Cu) (net 6))
+  (segment (start 216.9346 53.34) (end 219.71 56.1154) (width 0.6096) (layer F.Cu) (net 6))
+  (segment (start 204.47 53.34) (end 216.9346 53.34) (width 0.6096) (layer F.Cu) (net 6))
+  (segment (start 192.02 72.91) (end 193.79 72.91) (width 0.6096) (layer F.Cu) (net 6))
+  (segment (start 193.79 72.91) (end 194.31 72.39) (width 0.6096) (layer F.Cu) (net 6))
+  (segment (start 194.31 65.015) (end 194.555 64.77) (width 0.6096) (layer F.Cu) (net 6))
+  (segment (start 192.795 68.58) (end 193.04 68.58) (width 0.6096) (layer F.Cu) (net 6))
+  (segment (start 193.04 68.58) (end 194.31 67.31) (width 0.6096) (layer F.Cu) (net 6))
+  (segment (start 194.31 67.31) (end 194.31 65.015) (width 0.6096) (layer F.Cu) (net 6))
+  (segment (start 194.31 72.39) (end 194.31 67.31) (width 0.6096) (layer F.Cu) (net 6))
   (via (at 219.71 64.77) (size 0.8) (drill 0.4) (layers F.Cu B.Cu) (net 7))
   (via (at 219.71 59.69) (size 0.8) (drill 0.4) (layers F.Cu B.Cu) (net 7))
@@
   (segment (start 231.14 73.66) (end 229.09 73.66) (width 0.6096) (layer F.Cu) (net 7))
   (segment (start 226.84 71.9) (end 227.33 71.9) (width 0.6096) (layer F.Cu) (net 7))
-  (segment (start 219.71 64.77) (end 226.84 71.9) (width 0.6096) (layer F.Cu) (net 7))
   (segment (start 219.71 59.69) (end 219.71 64.77) (width 0.6096) (layer B.Cu) (net 7))
   (segment (start 217.71 57.69) (end 217.71 57.15) (width 0.6096) (layer F.Cu) (net 7))
@@
   (segment (start 234.06 90.63) (end 235.348 90.63) (width 0.25) (layer F.Cu) (net 7))
   (segment (start 232.33 88.9) (end 234.06 90.63) (width 0.25) (layer F.Cu) (net 7))
+  (segment (start 227.33 71.9) (end 221.76 71.9) (width 0.6096) (layer F.Cu) (net 7))
+  (segment (start 219.71 69.85) (end 219.71 64.77) (width 0.6096) (layer F.Cu) (net 7))
+  (segment (start 221.76 71.9) (end 219.71 69.85) (width 0.6096) (layer F.Cu) (net 7))
   (segment (start 243.06 71.9) (end 236.22 71.9) (width 0.6096) (layer F.Cu) (net 8))
   (segment (start 245.11 69.85) (end 243.06 71.9) (width 0.6096) (layer F.Cu) (net 8))
@@
   (segment (start 202.369999 118.549999) (end 203.2 119.38) (width 0.25) (layer F.Cu) (net 21))
   (via (at 203.2 119.38) (size 0.8) (drill 0.4) (layers F.Cu B.Cu) (net 21))
-  (via (at 232.41 121.92) (size 0.8) (drill 0.4) (layers F.Cu B.Cu) (net 21))
   (segment (start 205.74 115.325) (end 205.74 115.57) (width 0.25) (layer B.Cu) (net 21))
-  (segment (start 205.74 121.92) (end 204.47 120.65) (width 0.25) (layer B.Cu) (net 21))
-  (segment (start 218.44 121.92) (end 205.74 121.92) (width 0.25) (layer B.Cu) (net 21))
-  (segment (start 219.71 123.19) (end 218.44 121.92) (width 0.25) (layer B.Cu) (net 21))
   (segment (start 204.47 116.595) (end 205.74 115.325) (width 0.25) (layer B.Cu) (net 21))
   (segment (start 204.47 120.65) (end 204.47 116.595) (width 0.25) (layer B.Cu) (net 21))
   (segment (start 204.47 120.65) (end 203.2 119.38) (width 0.25) (layer B.Cu) (net 21))
-  (segment (start 231.14 123.19) (end 232.41 121.92) (width 0.25) (layer B.Cu) (net 21))
-  (segment (start 229.87 123.19) (end 231.14 123.19) (width 0.25) (layer B.Cu) (net 21))
-  (segment (start 229.87 123.19) (end 219.71 123.19) (width 0.25) (layer B.Cu) (net 21))
-  (segment (start 231.29 121.92) (end 232.41 121.92) (width 0.25) (layer F.Cu) (net 21))
-  (segment (start 230.02 120.65) (end 231.29 121.92) (width 0.25) (layer F.Cu) (net 21))
+  (segment (start 205.74 121.92) (end 222.25 121.92) (width 0.25) (layer B.Cu) (net 21))
+  (segment (start 222.25 121.92) (end 223.52 120.65) (width 0.25) (layer B.Cu) (net 21))
+  (segment (start 204.47 120.65) (end 205.74 121.92) (width 0.25) (layer B.Cu) (net 21))
   (segment (start 192.02 79.76) (end 191.77 80.01) (width 0.25) (layer F.Cu) (net 22))
   (segment (start 192.02 75.91) (end 192.02 79.76) (width 0.25) (layer F.Cu) (net 22))
-  (segment (start 190.745 70.135) (end 192.02 71.41) (width 0.25) (layer F.Cu) (net 23))
-  (segment (start 190.745 68.58) (end 190.745 70.135) (width 0.25) (layer F.Cu) (net 23))
+  (segment (start 190.745 70.135) (end 192.02 71.41) (width 0.6096) (layer F.Cu) (net 23))
+  (segment (start 190.745 68.58) (end 190.745 70.135) (width 0.6096) (layer F.Cu) (net 23))
   (segment (start 196.370001 94.772821) (end 195.58 93.98282) (width 0.25) (layer F.Cu) (net 24))
   (segment (start 196.370001 95.9612) (end 196.370001 94.772821) (width 0.25) (layer F.Cu) (net 24))
