File: ECE477.sch (KiCad schematic (older format))
At the start: 47 parts, among them IC1 LP3852EMP-3.3_NOPB, IC2 BQ29330DBT, J1 P7805-2000-S, J2 Conn_01x05_Male, J3 Conn_01x05_Male, J4 Conn_01x05_Male, J5 Conn_01x05_Male, J6 Conn_01x05_Male, J7 Conn_01x05_Male, SW1 SW_Push_Dual, U1 STM32H7_LQFP144_T2

Commit message: Added additional outputs on GPIOE
Parts:
- added H1, H2, H3, H4: MountingHole, MountingHole:MountingHole_3.2mm_M3_ISO14580, symbol Mechanical:MountingHole
- added J8: Conn_01x05_Male, Connector_PinHeader_2.54mm:PinHeader_1x06_P2.54mm_Vertical, symbol Connector:Conn_01x06_Male
Connections:
- net PIN1: now reaches U1.58 (PE8)
- net PIN1: now also J8.6 (Pin_6)
- net PIN2: now reaches U1.59 (PE9)
- net PIN2: now also J8.5 (Pin_5)
- net PIN3: now reaches U1.60 (PE10)
- net PIN3: now also J8.4 (Pin_4)
- net PIN4: now reaches U1.61 (PE11)
- net PIN4: now also J8.3 (Pin_3)
- net PIN5: now reaches U1.62 (PE12)
- net PIN5: now also J8.2 (Pin_2)
- net PIN6: now reaches U1.63 (PE13)
- net PIN6: now also J8.1 (Pin_1)
- no-connect marks 93 -> 87
Other:
- note removed: "WDI goes to CLK and LEDOUT goes to LEDPWR\n"
- moved on the sheet: C15, C16, C17, C18, C19, R7
